Commit message: added rotters

File: models/ingenuity_helicopter/urdf/helicopter.xacro (robot description, xacro)
@@ -4,5 +4,5 @@
     <link name="base_link"></link>
     <link name="helicopter_body">
-        <collision>
+       <collision>
             <origin xyz="0 0 0" rpy="0 0 0"></origin>
             <geometry>
@@ -20,9 +20,63 @@
         <inertial>
             <origin xyz="0 0 0"
-                rpy="0 0 0" />
+                 rpy="0 0 0" />
             <mass value="1.8" />
             <inertia ixx="2.56" ixy="0" ixz="0" iyy="2.56" iyz="0" izz="2.56"/>
         </inertial>
     </link>
+    <link name="propellor_1">
+        <collision>
+            <origin xyz="0 0 0" rpy="0 0 0"></origin>
+            <geometry>
+                <mesh filename="package://simulation/models/ingenuity_helicopter/meshes/propellor_1.dae"
+                    scale="1 1 1" />
+            </geometry>
+        </collision>
+        <visual>
+            <origin xyz="0 0 0" rpy="0 0 0"></origin>
+            <geometry>
+                <mesh filename="package://simulation/models/ingenuity_helicopter/meshes/propellor_1.dae"
+                    scale="1 1 1" />
+            </geometry>
+        </visual>
+        <inertial>
+            <origin xyz="0 0 0"
+                 rpy="0 0 0" />
+            <mass value="1.8" />
+            <inertia ixx="0.42" ixy="0" ixz="0" iyy="0.42" iyz="0" izz="0.42"/>
+        </inertial>
+    </link>
+    <link name="propellor_2">
+        <collision>
+            <origin xyz="0 0 0" rpy="0 0 0"></origin>
+            <geometry>
+                <mesh filename="package://simulation/models/ingenuity_helicopter/meshes/propellor-2.dae"
+                    scale="1 1 1" />
+            </geometry>
+        </collision>
+        <visual>
+            <origin xyz="0 0 0" rpy="0 0 0"></origin>
+            <geometry>
+                <mesh filename="package://simulation/models/ingenuity_helicopter/meshes/propellor-2.dae"
+                    scale="1 1 1" />
+            </geometry>
+        </visual>
+        <inertial>
+            <origin xyz="0 0 0"
+                 rpy="0 0 0" />
+            <mass value="1.8" />
+            <inertia ixx="0.42" ixy="0" ixz="0" iyy="0.42" iyz="0" izz="0.42"/>
+        </inertial>
+    </link>
+    <joint name="helicopter_body_propellor_1" type="fixed">
+        <parent link="helicopter_body"/>
+        <child link="propellor_1"/>
+        <origin rpy="0 0 0" xyz="-0.345 -0.435 0.4"/>
+    </joint>
+    <joint name="helicopter_body_propellor_2" type="fixed">
+        <parent link="helicopter_body"/>
+        <child link="propellor_2"/>
+        <origin rpy="0 0 0" xyz="0.9 0.35 1.03"/>
+    </joint>
     <joint name="base_link_helicopter_body" type="fixed">
         <parent link="base_link"/>

Commit message: add imu sensor

File: models/ingenuity_helicopter/urdf/helicopter.xacro (robot description, xacro)
@@ -4,5 +4,5 @@
     <link name="base_link"></link>
     <link name="helicopter_body">
-       <collision>
+        <collision>
             <origin xyz="0 0 0" rpy="0 0 0"></origin>
             <geometry>
@@ -20,14 +20,15 @@
         <inertial>
             <origin xyz="0 0 0"
-                 rpy="0 0 0" />
+                rpy="0 0 0" />
             <mass value="1.8" />
-            <inertia ixx="2.56" ixy="0" ixz="0" iyy="2.56" iyz="0" izz="2.56"/>
+            <inertia ixx="2.56" ixy="0" ixz="0" iyy="2.56" iyz="0" izz="2.56" />
         </inertial>
     </link>
-    <link name="propellor_1">
+    <link name="propellor_up">
         <collision>
             <origin xyz="0 0 0" rpy="0 0 0"></origin>
             <geometry>
-                <mesh filename="package://simulation/models/ingenuity_helicopter/meshes/propellor_1.dae"
+                <mesh
+                    filename="package://simulation/models/ingenuity_helicopter/meshes/rotor_up.dae"
                     scale="1 1 1" />
             </geometry>
@@ -36,5 +37,6 @@
             <origin xyz="0 0 0" rpy="0 0 0"></origin>
             <geometry>
-                <mesh filename="package://simulation/models/ingenuity_helicopter/meshes/propellor_1.dae"
+                <mesh
+                    filename="package://simulation/models/ingenuity_helicopter/meshes/rotor_up.dae"
                     scale="1 1 1" />
             </geometry>
@@ -42,14 +44,15 @@
         <inertial>
             <origin xyz="0 0 0"
-                 rpy="0 0 0" />
+                rpy="0 0 0" />
             <mass value="1.8" />
-            <inertia ixx="0.42" ixy="0" ixz="0" iyy="0.42" iyz="0" izz="0.42"/>
+            <inertia ixx="0.42" ixy="0" ixz="0" iyy="0.42" iyz="0" izz="0.42" />
         </inertial>
     </link>
-    <link name="propellor_2">
+    <link name="propellor_down">
         <collision>
             <origin xyz="0 0 0" rpy="0 0 0"></origin>
             <geometry>
-                <mesh filename="package://simulation/models/ingenuity_helicopter/meshes/propellor-2.dae"
+                <mesh
+                    filename="package://simulation/models/ingenuity_helicopter/meshes/rotor_down.dae"
                     scale="1 1 1" />
             </geometry>
@@ -58,5 +61,6 @@
             <origin xyz="0 0 0" rpy="0 0 0"></origin>
             <geometry>
-                <mesh filename="package://simulation/models/ingenuity_helicopter/meshes/propellor-2.dae"
+                <mesh
+                    filename="package://simulation/models/ingenuity_helicopter/meshes/rotor_down.dae"
                     scale="1 1 1" />
             </geometry>
@@ -64,18 +68,22 @@
         <inertial>
             <origin xyz="0 0 0"
-                 rpy="0 0 0" />
+                rpy="0 0 0" />
             <mass value="1.8" />
-            <inertia ixx="0.42" ixy="0" ixz="0" iyy="0.42" iyz="0" izz="0.42"/>
+            <inertia ixx="0.42" ixy="0" ixz="0" iyy="0.42" iyz="0" izz="0.42" />
         </inertial>
     </link>
-    <joint name="helicopter_body_propellor_1" type="fixed">
-        <parent link="helicopter_body"/>
-        <child link="propellor_1"/>
-        <origin rpy="0 0 0" xyz="-0.345 -0.435 0.4"/>
+    <joint name="body_propellor_up_joint" type="continuous">
+        <parent link="helicopter_body" />
+        <child link="propellor_up" />
+        <origin rpy="0 0 0" xyz="0 0 0.46" /> <!-- xyz="-0.345 -0.435 0.40"-->
+        <axis xyz="0 0 1" />
+        <dynamics damping="0.0" friction="0.0" />
     </joint>
-    <joint name="helicopter_body_propellor_2" type="fixed">
-        <parent link="helicopter_body"/>
-        <child link="propellor_2"/>
-        <origin rpy="0 0 0" xyz="0.9 0.35 1.03"/>
+    <joint name="body_propellor_down_joint" type="continuous">
+        <parent link="helicopter_body" />
+        <child link="propellor_down" />
+        <origin rpy="0 0 0" xyz="0 0 0.35" />
+        <axis xyz="0 0 1" />
+        <dynamics damping="0.0" friction="0.0" />
     </joint>
     <joint name="base_link_helicopter_body" type="fixed">
@@ -83,3 +91,23 @@
         <child link="helicopter_body"/>
     </joint>
+    <transmission name="helicopter_body_propellor_up_trans">
+        <type>transmission_interface/SimpleTransmission</type>
+        <joint name="body_propellor_up_joint">
+            <hardwareInterface>hardware_interface/VelocityJointInterface</hardwareInterface>
+        </joint>
+        <actuator name="propellor_up_motor">
+            <hardwareInterface>hardware_interface/EffortJointInterface</hardwareInterface>
+            <mechanicalReduction>1</mechanicalReduction>
+        </actuator>
+    </transmission>
+    <transmission name="helicopter_body_propellor_down_trans">
+        <type>transmission_interface/SimpleTransmission</type>
+        <joint name="body_propellor_down_joint">
+            <hardwareInterface>hardware_interface/VelocityJointInterface</hardwareInterface>
+        </joint>
+        <actuator name="propellor_down_motor">
+            <hardwareInterface>hardware_interface/EffortJointInterface</hardwareInterface>
+            <mechanicalReduction>1</mechanicalReduction>
+        </actuator>
+    </transmission>
 </robot>

Commit message: configure imu sensor and attached to the body

File: models/ingenuity_helicopter/urdf/helicopter.xacro (robot description, xacro)
@@ -76,5 +76,5 @@
         <parent link="helicopter_body" />
         <child link="propellor_up" />
-        <origin rpy="0 0 0" xyz="0 0 0.46" /> <!-- xyz="-0.345 -0.435 0.40"-->
+        <origin rpy="0 0 0" xyz="0 0 0.46" />
         <axis xyz="0 0 1" />
         <dynamics damping="0.0" friction="0.0" />

Commit message: added liftdrag plugin

File: models/ingenuity_helicopter/urdf/helicopter.xacro (robot description, xacro)
@@ -2,5 +2,18 @@
 <robot name="helicopter" xmlns:xacro="http://www.ros.org/wiki/xacro">
     <xacro:include filename="$(find simulation)/models/ingenuity_helicopter/urdf/helicopter.gazebo" />
-    <link name="base_link"></link>
+    <link name="base_link_footprint">
+    </link>
+    <link name="base_link">
+        <inertial>
+            <origin xyz="0 0 0"
+                rpy="0 0 0" />
+            <mass value="1.8" />
+            <inertia ixx="1.66" ixy="0" ixz="0" iyy="1.66" iyz="0" izz="2.56" />
+        </inertial>
+    </link>
+    <joint name="base_footprint_base_link_joint" type="fixed">
+        <parent link="base_link_footprint"/>
+        <child link="base_link"/>
+    </joint>
     <link name="helicopter_body">
         <collision>
@@ -87,7 +100,9 @@
         <dynamics damping="0.0" friction="0.0" />
     </joint>
-    <joint name="base_link_helicopter_body" type="fixed">
+    <joint name="base_link_body_joint" type="continuous">
         <parent link="base_link"/>
         <child link="helicopter_body"/>
+        <origin rpy="0 0 0" xyz="0 0 0" />
+        <axis xyz="0 0 1" />
     </joint>
     <transmission name="helicopter_body_propellor_up_trans">

Commit message: add fixed mount link

File: models/ingenuity_helicopter/urdf/helicopter.xacro (robot description, xacro)
@@ -2,18 +2,5 @@
 <robot name="helicopter" xmlns:xacro="http://www.ros.org/wiki/xacro">
     <xacro:include filename="$(find simulation)/models/ingenuity_helicopter/urdf/helicopter.gazebo" />
-    <link name="base_link_footprint">
-    </link>
-    <link name="base_link">
-        <inertial>
-            <origin xyz="0 0 0"
-                rpy="0 0 0" />
-            <mass value="1.8" />
-            <inertia ixx="1.66" ixy="0" ixz="0" iyy="1.66" iyz="0" izz="2.56" />
-        </inertial>
-    </link>
-    <joint name="base_footprint_base_link_joint" type="fixed">
-        <parent link="base_link_footprint"/>
-        <child link="base_link"/>
-    </joint>
+    <link name="base_link"></link>
     <link name="helicopter_body">
         <collision>
@@ -100,9 +87,9 @@
         <dynamics damping="0.0" friction="0.0" />
     </joint>
-    <joint name="base_link_body_joint" type="continuous">
+    <joint name="base_link_body_joint" type="fixed">
         <parent link="base_link"/>
         <child link="helicopter_body"/>
-        <origin rpy="0 0 0" xyz="0 0 0" />
-        <axis xyz="0 0 1" />
+        <origin xyz="0 0 0" rpy="0 0 0"/>
+		<axis xyz="0 0 1" />
     </joint>
     <transmission name="helicopter_body_propellor_up_trans">
